File: UINIO-Cubic-Prism.kicad_pcb (KiCad board)
At the start: 2 copper layers, 87.2 x 35.9 mm, 53 parts, among them Q1 AO3415A, Q2 AO3415A, U1 CP2102, U10 ME6211, U11 RGB_WS2812B_5050, U12 FPC-SMD_8P-0.5mm, U13 AMS1117, U14 CON_12Pin, U2 BH1750FVI, U3 FPC-SMD_8P-0.5mm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

Commit message: Release UINIO-Cubic-Prism version 3.0.0.
Parts:
- removed the ? at (149.0, 109.8)
- removed the ? at (154.6, 78.1)
- added ?: LOGO, LOGO, F.Cu at (149.1, 109.7)
Other:
- outline, holes or cut-outs redrawn
- board text added: "UINIO-Cubic-Prism"
- board text added: "Version 3.0.0"
- board text removed: "CUBIC"
- board text removed: "UINIO"
- board text removed: "Version 2.0.0"
