File: UINIO-Cubic-Prism.kicad_sch (KiCad schematic)
At the start: 45 parts, among them Q1 AO3415A, Q2 AO3415A, U1 CP2102, U10 ME6211, U11 RGB_WS2812B_5050, U12 FPC-SMD_8P-0.5mm, U13 AMS1117, U14 CON_12Pin, U2 BH1750FVI, U3 FPC-SMD_8P-0.5mm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

Commit message: Release UINIO-Cubic-Prism version 3.0.0.
Other:
- company: Hank -> 电子技术博客 UinIO.com
Changed lines of the file:
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@@
   (title_block
     (title "UINIO-Cubic-Prism")
-    (date "2022-10-26")
-    (rev "UinIO.com")
-    (company "Hank")
+    (date "2023-01-29")
+    (rev "Version 3.0.0")
+    (company "电子技术博客 UinIO.com")
   )
   (junction (at 287.274 122.428) (diameter 0) (color 0 0 0 0)
